File: KiCad/ya_brakeboardESP32_S3/MCP.kicad_sch (KiCad schematic)
At the start: 7 parts, among them J5 I2C0_Terminal, J6 MCP#0_Terminal, J7 MCP#1_Terminal, J8 MCP#2_Terminal, U4 MCP23017_SP, U5 MCP23017_SP, U6 MCP23017_SP

Commit message: basic schematics finished
Parts:
- removed J5: I2C0_Terminal, symbol Connector:Screw_Terminal_01x08
- removed J6: MCP#0_Terminal, symbol Connector:Screw_Terminal_01x16
- removed J7: MCP#1_Terminal, symbol Connector:Screw_Terminal_01x16
- removed J8: MCP#2_Terminal, symbol Connector:Screw_Terminal_01x16
- removed U6: MCP23017_SP, Package_DIP:DIP-28_W7.62mm, symbol Interface_Expansion:MCP23017_SP
- added R1, R2: 100k, symbol Device:R_Small
Connections:
- net +3V3: now also R1.2, R2.2
- net SDA_0: now reaches U4.13 (SDA), U5.13 (SDA)
- net SDA_0: no longer U5.12 (SCK)
- net X_INPOS: now reaches U5.1 (GPB0)
- net at U5.18 (~{RESET}): now also R2.1
- net GPIO_MCP1_INTB: now reaches U5.19 (INTB)
- net Y_INPOS: now reaches U5.2 (GPB1)
- net GPIO_MCP1_INTA: now reaches U5.20 (INTA)
- net X_ALARM_INPUT: now reaches U5.21 (GPA0)
- net Y_ALARM_INPUT: now reaches U5.22 (GPA1)
- net Z_ALARM_INPUT: now reaches U5.23 (GPA2)
- net A_ALARM_INPUT: now reaches U5.24 (GPA3)
- net B_ALARM_INPUT: now reaches U5.25 (GPA4)
- net C_ALARM_INPUT: now reaches U5.26 (GPA5)
- net D_ALARM_INPUT: now reaches U5.27 (GPA6)
- net GP_IN_0: now reaches U5.28 (GPA7)
- net Z_INPOS: now reaches U5.3 (GPB2)
- net A_INPOS: now reaches U5.4 (GPB3)
- net B_INPOS: now reaches U5.5 (GPB4)
- net GP_IN_1: now reaches U5.6 (GPB5)
- net GP_IN_2: now reaches U5.7 (GPB6)
- net GP_IN_3: now reaches U5.8 (GPB7)
- net B_LIMIT_MIN: now reaches U4.1 (GPB0)
- net X_LIMIT_MAX: now reaches U4.22 (GPA1)
- net Y_LIMIT_MIN: now reaches U4.23 (GPA2)
- net Y_LIMIT_MAX: now reaches U4.24 (GPA3)
- net Z_LIMIT_MIN: now reaches U4.25 (GPA4)
- net Z_LIMIT_MAX: now reaches U4.26 (GPA5)
- net A_LIMIT_MIN: now reaches U4.27 (GPA6)
- net A_LIMIT_MAX: now reaches U4.28 (GPA7)
- net B_LIMIT_MAX: now reaches U4.2 (GPB1)
- net C_LIMIT_MIN: now reaches U4.3 (GPB2)
- net C_LIMIT_MAX: now reaches U4.4 (GPB3)
- net D_LIMIT_MIN: now reaches U4.5 (GPB4)
- net D_LIMIT_MAX: now reaches U4.6 (GPB5)
- net E_LIMIT_MIN: now reaches U4.7 (GPB6)
- net E_LIMIT_MAX: now reaches U4.8 (GPB7)
- net X_LIMIT_MIN: now reaches U4.21 (GPA0)
- net SCK_0: now reaches U4.12 (SCK)
- net SCK_0: now also U5.12 (SCK)
- net GPIO_MCP0_INTB: now reaches U4.19 (INTB)
- net GPIO_MCP0_INTA: now reaches U4.20 (INTA)
- net at U4.18 (~{RESET}): now also R1.1
