File: KiCad/ya_brakeboardESP32_S3/shift_registers.kicad_sch (KiCad schematic)
At the start: 15 parts, among them U1 TPIC6B595N, U2 TPIC6B595N, U3 TPIC6B595N, U7 TPIC6B595N, U8 TPIC6B595N

Commit message: ready for implementation
Connections:
- net SR_CLCK renamed SRCK
- net SR_CS renamed RCK
- net SR_MOSI renamed SERIN
- net SR_OE renamed G
Changed lines of the file:
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@@
 		)
 	)
-	(hierarchical_label "SR_CS"
+	(hierarchical_label "RCK"
 		(shape input)
 		(at 36.83 53.34 180)
@@
 		)
 	)
-	(hierarchical_label "SR_OE"
+	(hierarchical_label "G"
 		(shape input)
 		(at 36.83 50.8 180)
@@
 		)
 	)
-	(hierarchical_label "SR_CLCK"
+	(hierarchical_label "SRCK"
 		(shape input)
 		(at 36.83 58.42 180)
@@
 		)
 	)
-	(hierarchical_label "SR_MOSI"
+	(hierarchical_label "SERIN"
 		(shape input)
 		(at 36.83 55.88 180)
